File: without_ground_holes.kicad_pcb (KiCad board)
At the start: 2 copper layers, 59 parts, among them J1 COAX, J2 Qwicc_6-pin, U1 SKY67013-396LF_CID141, U2 SX1272IMLTRICT-ND_CID104, U3 SKY67013-396LF_CID141, U4 PE4259_CID105, U5 ATMEGA328P-AU, X1 X1E0000210162_CID142, X2 7A-12.000MAAJ-T_CID117

Commit message: PCB finished
Parts:
- added ?: , dtusat:via-0.6mm-0.3mm_drill, F.Cu at (48.9, 31.4)
- added ?: , dtusat:via-0.6mm-0.3mm_drill, F.Cu at (50.9, 35.4)
- added ?: , dtusat:via-0.6mm-0.3mm_drill, F.Cu at (51.9, 35.4)
- added ?: , dtusat:via-0.6mm-0.3mm_drill, F.Cu at (53.0, 35.4)
- added ?: , dtusat:via-0.6mm-0.3mm_drill, F.Cu at (54.0, 35.0)
- added ?: , dtusat:via-0.6mm-0.3mm_drill, F.Cu at (53.9, 36.1)
- added ?: , dtusat:via-0.6mm-0.3mm_drill, F.Cu at (53.7, 37.1)
- added ?: , dtusat:via-0.6mm-0.3mm_drill, F.Cu at (52.6, 37.1)
- added ?: , dtusat:via-0.6mm-0.3mm_drill, F.Cu at (51.6, 37.1)
- added ?: , dtusat:via-0.6mm-0.3mm_drill, F.Cu at (51.1, 38.0)
- added ?: , dtusat:via-0.6mm-0.3mm_drill, F.Cu at (50.0, 37.9)
- added ?: , dtusat:via-0.6mm-0.3mm_drill, F.Cu at (48.0, 30.5)
- added ?: , dtusat:via-0.6mm-0.3mm_drill, F.Cu at (49.0, 37.9)
- added ?: , dtusat:via-0.6mm-0.3mm_drill, F.Cu at (48.3, 37.1)
- added ?: , dtusat:via-0.6mm-0.3mm_drill, F.Cu at (47.2, 37.2)
- added ?: , dtusat:via-0.6mm-0.3mm_drill, F.Cu at (46.5, 37.8)
- added ?: , dtusat:via-0.6mm-0.3mm_drill, F.Cu at (45.5, 38.4)
- added ?: , dtusat:via-0.6mm-0.3mm_drill, F.Cu at (45.5, 37.4)
- added ?: , dtusat:via-0.6mm-0.3mm_drill, F.Cu at (45.5, 36.3)
- added ?: , dtusat:via-0.6mm-0.3mm_drill, F.Cu at (45.5, 35.3)
- added ?: , dtusat:via-0.6mm-0.3mm_drill, F.Cu at (45.9, 34.4)
- added ?: , dtusat:via-0.6mm-0.3mm_drill, F.Cu at (46.1, 33.4)
- added ?: , dtusat:via-0.6mm-0.3mm_drill, F.Cu at (52.0, 32.1)
- added ?: , dtusat:via-0.6mm-0.3mm_drill, F.Cu at (46.1, 32.3)
- added ?: , dtusat:via-0.6mm-0.3mm_drill, F.Cu at (42.9, 42.4)
- added ?: , dtusat:via-0.6mm-0.3mm_drill, F.Cu at (46.6, 41.2)
- added ?: , dtusat:via-0.6mm-0.3mm_drill, F.Cu at (45.9, 31.3)
- added ?: , dtusat:via-0.6mm-0.3mm_drill, F.Cu at (46.6, 40.2)
- added ?: , dtusat:via-0.6mm-0.3mm_drill, F.Cu at (47.7, 39.9)
- added ?: , dtusat:via-0.6mm-0.3mm_drill, F.Cu at (48.7, 40.0)
- added ?: , dtusat:via-0.6mm-0.3mm_drill, F.Cu at (49.8, 40.0)
- added ?: , dtusat:via-0.6mm-0.3mm_drill, F.Cu at (41.2, 36.9)
- added ?: , dtusat:via-0.6mm-0.3mm_drill, F.Cu at (40.8, 38.9)
- added ?: , dtusat:via-0.6mm-0.3mm_drill, F.Cu at (49.8, 32.4)
- added ?: , dtusat:via-0.6mm-0.3mm_drill, F.Cu at (41.8, 38.6)
- added ?: , dtusat:via-0.6mm-0.3mm_drill, F.Cu at (42.8, 38.6)
- added ?: , dtusat:via-0.6mm-0.3mm_drill, F.Cu at (43.5, 37.8)
- added ?: , dtusat:via-0.6mm-0.3mm_drill, F.Cu at (43.5, 36.8)
- added ?: , dtusat:via-0.6mm-0.3mm_drill, F.Cu at (43.5, 35.8)
- added ?: , dtusat:via-0.6mm-0.3mm_drill, F.Cu at (42.6, 35.4)
- added ?: , dtusat:via-0.6mm-0.3mm_drill, F.Cu at (42.6, 34.4)
- added ?: , dtusat:via-0.6mm-0.3mm_drill, F.Cu at (42.9, 33.4)
- added ?: , dtusat:via-0.6mm-0.3mm_drill, F.Cu at (42.9, 32.4)
- added ?: , dtusat:via-0.6mm-0.3mm_drill, F.Cu at (42.6, 31.4)
- added ?: , dtusat:via-0.6mm-0.3mm_drill, F.Cu at (48.3, 32.6)
- added ?: , dtusat:via-0.6mm-0.3mm_drill, F.Cu at (43.1, 30.6)
- added ?: , dtusat:via-0.6mm-0.3mm_drill, F.Cu at (44.2, 30.6)
- added ?: , dtusat:via-0.6mm-0.3mm_drill, F.Cu at (45.0, 30.0)
- added ?: , dtusat:via-0.6mm-0.3mm_drill, F.Cu at (46.9, 34.2)
- added ?: , dtusat:via-0.6mm-0.3mm_drill, F.Cu at (47.9, 34.5)
- added ?: , dtusat:via-0.6mm-0.3mm_drill, F.Cu at (49.0, 34.5)
- added ?: , dtusat:via-0.6mm-0.3mm_drill, F.Cu at (50.0, 34.8)
- L2: value L_0402_33nH_CID3034 -> L0402
- moved C31 85.3 mm to (69.4, 30.7)
- moved R4 85.3 mm to (75.5, 38.3)
- moved C32 85.3 mm to (69.7, 34.5)
- moved C33 85.3 mm to (69.7, 38.3)
- moved C34 85.3 mm to (69.7, 42.1)
- moved C35 85.3 mm to (69.7, 45.7)
- moved C36 85.3 mm to (69.7, 49.7)
- moved X2 44.1 mm to (64.0, 68.9)
Connections:
- C1 pad 2: GND -> Net-(C1-Pad2)
- L2 pad 2: Net-(L2-Pad2) -> (no net)
- U5 pad 32: /RXTX_SW -> /ResetSX
Routing:
- net +3V3: track 82.6 -> 105.9 mm
- net Net-(C2-Pad1): track 0.00 -> 8.24 mm
