File: LoRa_FR4_1/LoRa_Balloon.kicad_pcb (KiCad board)
At the start: 2 copper layers, 30 x 56 mm, 253 parts, among them J2 Qwicc_6-pin, U1 SKY67013-396LF_CID141, U2 SX1272IMLTRICT-ND_CID104, U3 SKY67013-396LF_CID141, U4 PE4259_CID105, U5 ATMEGA328P-AU, U6 XCL205, X1 X1E0000210162_CID142, X2 7A-12.000MAAJ-T_CID117

Commit message: New FR4 versions
Parts:
- added ?: , dtusat:via-0.6mm-0.3mm_drill, F.Cu at (124.0, 151.3)
- added ?: , dtusat:via-0.6mm-0.3mm_drill, F.Cu at (112.5, 104.0)
- added ?: , dtusat:via-0.6mm-0.3mm_drill, F.Cu at (111.5, 104.0)
- added ?: , dtusat:via-0.6mm-0.3mm_drill, F.Cu at (110.5, 104.0)
- added ?: , dtusat:via-0.6mm-0.3mm_drill, F.Cu at (109.5, 104.0)
- added ?: , dtusat:via-0.6mm-0.3mm_drill, F.Cu at (108.5, 104.0)
- added ?: , dtusat:via-0.6mm-0.3mm_drill, F.Cu at (107.8, 104.7)
- added ?: , dtusat:via-0.6mm-0.3mm_drill, F.Cu at (107.1, 105.4)
- added ?: , dtusat:via-0.6mm-0.3mm_drill, F.Cu at (106.4, 106.1)
- added ?: , dtusat:via-0.6mm-0.3mm_drill, F.Cu at (105.7, 106.8)
- added ?: , dtusat:via-0.6mm-0.3mm_drill, F.Cu at (105.0, 107.6)
- added ?: , dtusat:via-0.6mm-0.3mm_drill, F.Cu at (127.3, 147.4)
- added ?: , dtusat:via-0.6mm-0.3mm_drill, F.Cu at (119.5, 104.0)
- added ?: , dtusat:via-0.6mm-0.3mm_drill, F.Cu at (118.5, 104.0)
- added ?: , dtusat:via-0.6mm-0.3mm_drill, F.Cu at (117.5, 104.0)
- added ?: , dtusat:via-0.6mm-0.3mm_drill, F.Cu at (116.5, 104.0)
- added ?: , dtusat:via-0.6mm-0.3mm_drill, F.Cu at (115.5, 104.0)
- added ?: , dtusat:via-0.6mm-0.3mm_drill, F.Cu at (114.5, 104.0)
- added ?: , dtusat:via-0.6mm-0.3mm_drill, F.Cu at (113.5, 104.0)
- added J1: Qwiic_4pin, dtusat:Qwiic_4-pin, F.Cu at (127.6, 147.3)
- A1: moved to F.Cu
- moved F1 89.9 mm to (102.6, 110.1)
- moved ? 87.1 mm to (121.2, 150.6)
- moved ? 87.0 mm to (121.2, 152.6)
- moved H1 85.9 mm to (102.1, 140.5)
- moved ? 85.8 mm to (111.4, 112.8)
- moved ? 85.8 mm to (121.1, 157.4)
- moved ? 85.8 mm to (109.5, 124.6)
- moved ? 85.8 mm to (109.9, 142.8)
- moved ? 85.8 mm to (118.0, 116.5)
- moved ? 85.8 mm to (119.9, 117.0)
- moved ? 85.8 mm to (109.8, 151.8)
- moved ? 85.8 mm to (111.4, 151.8)
- moved ? 85.8 mm to (106.5, 118.0)
- moved ? 85.8 mm to (126.9, 137.6)
- moved ? 85.8 mm to (123.5, 112.8)
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Connections:
- C10 pad 1: Net-(C10-Pad1) -> +3V3
- U2 pad 15: Net-(C10-Pad1) -> +3V3
Routing:
- net /RX: track 10.5 -> 28.5 mm, vias 0 -> 2
- net /TX: track 9.71 -> 27.7 mm, vias 0 -> 2
- net Net-(A1-Pad1): track 17.8 -> 23.4 mm, vias 1 -> 0
- net /RF_antenna: track 6.41 -> 10.1 mm
- net +3V3: track 187.4 -> 188.3 mm
Other:
- board size 30 x 56 mm -> 30 x 61 mm
