File: LoRa_FR4_2/LoRa_Balloon.kicad_pcb (KiCad board)
At the start: 2 copper layers, 30 x 56 mm, 253 parts, among them J2 Qwicc_6-pin, U1 SKY67013-396LF_CID141, U2 SX1272IMLTRICT-ND_CID104, U3 SKY67013-396LF_CID141, U4 PE4259_CID105, U5 ATMEGA328P-AU, U6 XCL205, X1 X1E0000210162_CID142, X2 7A-12.000MAAJ-T_CID117

Commit message: New FR4 versions
Parts:
- added ?: , dtusat:via-0.6mm-0.3mm_drill, F.Cu at (123.5, 153.5)
- added ?: , dtusat:via-0.6mm-0.3mm_drill, F.Cu at (112.5, 104.0)
- added ?: , dtusat:via-0.6mm-0.3mm_drill, F.Cu at (111.5, 104.0)
- added ?: , dtusat:via-0.6mm-0.3mm_drill, F.Cu at (110.5, 104.0)
- added ?: , dtusat:via-0.6mm-0.3mm_drill, F.Cu at (109.5, 104.0)
- added ?: , dtusat:via-0.6mm-0.3mm_drill, F.Cu at (108.5, 104.0)
- added ?: , dtusat:via-0.6mm-0.3mm_drill, F.Cu at (107.8, 104.7)
- added ?: , dtusat:via-0.6mm-0.3mm_drill, F.Cu at (107.1, 105.4)
- added ?: , dtusat:via-0.6mm-0.3mm_drill, F.Cu at (106.4, 106.1)
- added ?: , dtusat:via-0.6mm-0.3mm_drill, F.Cu at (105.7, 106.8)
- added ?: , dtusat:via-0.6mm-0.3mm_drill, F.Cu at (105.0, 107.6)
- added ?: , dtusat:via-0.6mm-0.3mm_drill, F.Cu at (123.6, 149.9)
- added ?: , dtusat:via-0.6mm-0.3mm_drill, F.Cu at (119.5, 104.0)
- added ?: , dtusat:via-0.6mm-0.3mm_drill, F.Cu at (118.5, 104.0)
- added ?: , dtusat:via-0.6mm-0.3mm_drill, F.Cu at (117.5, 104.0)
- added ?: , dtusat:via-0.6mm-0.3mm_drill, F.Cu at (116.5, 104.0)
- added ?: , dtusat:via-0.6mm-0.3mm_drill, F.Cu at (115.5, 104.0)
- added ?: , dtusat:via-0.6mm-0.3mm_drill, F.Cu at (114.5, 104.0)
- added ?: , dtusat:via-0.6mm-0.3mm_drill, F.Cu at (113.5, 104.0)
- added J1: Qwiic_4pin, dtusat:Qwiic_4-pin, F.Cu at (127.6, 147.1)
- A1: moved to B.Cu
- moved F1 89.9 mm to (102.6, 110.1)
- moved ? 87.1 mm to (121.2, 150.6)
- moved ? 87.0 mm to (121.2, 152.5)
- moved H1 85.9 mm to (102.1, 140.5)
- moved ? 85.8 mm to (111.4, 112.8)
- moved ? 85.8 mm to (121.1, 157.4)
- moved ? 85.8 mm to (109.5, 124.6)
- moved ? 85.8 mm to (109.9, 142.8)
- moved ? 85.8 mm to (118.0, 116.5)
- moved ? 85.8 mm to (119.9, 117.0)
- moved ? 85.8 mm to (109.8, 151.8)
- moved ? 85.8 mm to (111.4, 151.8)
- moved ? 85.8 mm to (106.5, 118.0)
- moved ? 85.8 mm to (126.9, 137.6)
- moved ? 85.8 mm to (123.5, 112.8)
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Connections:
- C10 pad 1: Net-(C10-Pad1) -> +3V3
- C2 pad 1: Net-(C10-Pad1) -> +3V3
- U2 pad 1: Net-(C10-Pad1) -> +3V3
- U2 pad 15: Net-(C10-Pad1) -> +3V3
Routing:
- net Net-(A1-Pad1): track 0.00 -> 23.4 mm, vias 0 -> 1
- net (no net): track 0.00 -> 20.3 mm
- net /RX: track 10.5 -> 30.4 mm, vias 0 -> 2
- net /TX: track 9.71 -> 29.6 mm, vias 0 -> 2
- net /RF_antenna: track 6.41 -> 10.1 mm
- net +3V3: track 187.4 -> 188.3 mm
- added copper zone on B.Cu, net GND
Other:
- board size 30 x 56 mm -> 30 x 61 mm
