File: LoRa Balloon Mk2.1/LoRa_Balloon.kicad_pcb (KiCad board)
At the start: 2 copper layers, 30 x 61 mm, 273 parts, among them J1 Qwiic_4pin, J2 Qwicc_6-pin, U1 SKY67013-396LF_CID141, U2 SX1272IMLTRICT-ND_CID104, U3 SKY67013-396LF_CID141, U4 PE4259_CID105, U5 ATMEGA328P-AU, U6 XCL205, X1 X1E0000210162_CID142, X2 7A-12.000MAAJ-T_CID117

Commit message: Updated libraries
Parts:
- moved U2 0.10 mm to (111.7, 132.3)
- turned F1 to 0 degrees
- turned U6 to 0 degrees
Connections:
- C2 pad 1: Net-(C10-Pad1) -> +3V3
- U2 pad 1: Net-(C10-Pad1) -> +3V3
- U6 pad GND: (no net) -> GND
Routing:
- net +3V3: track 188.3 -> 186.0 mm
- net Net-(L4-Pad2): track 0.00 -> 1.29 mm
Other:
- board text added: "JLCJLCJLCJLC"
