File: LoRa Balloon Mk3/LoRa_Balloon.kicad_pcb (KiCad board)
At the start: 2 copper layers, 30 x 47 mm, 203 parts, among them J2 Edge_connector_9_pin, U1 SKY67013-396LF_CID141, U2 SX1272IMLTRICT-ND_CID104, U3 SKY67013-396LF_CID141, U4 XCL205, U5 PE4259_CID105, U6 ATMEGA328P-MMH, U7 ublox_MAX-M8C, X1 X1E0000210162_CID142, X2 7A-12.000MAAJ-T_CID117

Commit message: Mk3 enclosure created
Other:
- board text added: "JLCJLCJLCJLC"
